Commit message: feat: アームを追加

File: src/sum2026_description/urdf/sum2026.urdf.xacro (robot description, xacro)
@@ -4,3 +4,9 @@
     <xacro:include filename="mobile_base.xacro" />
     <xacro:include filename="mobile_base.ros2_control.xacro" />
+    <xacro:include filename="arm.xacro" />
+    <joint name="mobile_base_arm_joint" type="fixed">
+        <parent link="base_link" />
+        <child link="arm_base_link" />
+        <origin xyz="${base_length / 4.0} 0 ${base_height}" rpy="0 0 0" />
+    </joint>
 </robot>
