Commit message: feat: LiDARを追加

File: src/sum2026_description/urdf/mobile_base.xacro (robot description, xacro)
@@ -6,4 +6,6 @@
     <xacro:property name="wheel_radius" value="0.1" />
     <xacro:property name="wheel_length" value="0.05" />
+    <xacro:property name="lidar_radius" value="0.05" />
+    <xacro:property name="lidar_height" value="0.06" />
     <link name="base_footprint" />
     <link name="base_link">
@@ -62,4 +64,23 @@
                               o_xyz="0 0 0" o_rpy="0 0 0" />
     </link>
+    <link name="lidar_link">
+        <visual>
+            <geometry>
+                <cylinder radius="${lidar_radius}" length="${lidar_height}" />
+            </geometry>
+            <origin xyz="0 0 ${lidar_height / 2.0}" rpy="0 0 0" />
+            <material name="green">
+                <color rgba="0 0.8 0 1" />
+            </material>
+        </visual>
+        <collision>
+            <geometry>
+                <cylinder radius="${lidar_radius}" length="${lidar_height}" />
+            </geometry>
+            <origin xyz="0 0 ${lidar_height / 2.0}" rpy="0 0 0" />
+        </collision>
+        <xacro:cylinder_inertia m="0.2" r="${lidar_radius}" l="${lidar_height}"
+                                o_xyz="0 0 ${lidar_height / 2.0}" o_rpy="0 0 0" />
+    </link>
     <joint name="base_joint" type="fixed">
         <parent link="base_footprint" />
@@ -84,3 +105,8 @@
         <origin xyz="${base_length / 3.0} 0 ${-wheel_radius / 2.0}" rpy="0 0 0" />
     </joint>
+    <joint name="base_lidar_joint" type="fixed">
+        <parent link="base_link" />
+        <child link="lidar_link" />
+        <origin xyz="0 0 ${base_height}" rpy="0 0 0" />
+    </joint>
 </robot>

File: src/sum2026_description/urdf/sum2026.urdf.xacro (robot description, xacro)
@@ -24,4 +24,27 @@
             <mu2 value="0.1" />
         </gazebo>
+        <gazebo reference="lidar_link">
+            <sensor name="lidar" type="gpu_lidar">
+                <topic>scan</topic>
+                <update_rate>10</update_rate>
+                <lidar>
+                    <scan>
+                        <horizontal>
+                            <samples>360</samples>
+                            <resolution>1</resolution>
+                            <min_angle>-${pi}</min_angle>
+                            <max_angle>${pi}</max_angle>
+                        </horizontal>
+                    </scan>
+                    <range>
+                        <min>0.12</min>
+                        <max>10.0</max>
+                        <resolution>0.01</resolution>
+                    </range>
+                </lidar>
+                <always_on>true</always_on>
+                <visualize>true</visualize>
+            </sensor>
+        </gazebo>
         <gazebo>
             <plugin filename="gz_ros2_control-system" name="gz_ros2_control::GazeboSimROS2ControlPlugin">

Commit message: feat: lidar.xacroに分離

File: src/sum2026_description/urdf/mobile_base.xacro (robot description, xacro)
@@ -6,6 +6,4 @@
     <xacro:property name="wheel_radius" value="0.1" />
     <xacro:property name="wheel_length" value="0.05" />
-    <xacro:property name="lidar_radius" value="0.05" />
-    <xacro:property name="lidar_height" value="0.06" />
     <link name="base_footprint" />
     <link name="base_link">
@@ -64,23 +62,4 @@
                               o_xyz="0 0 0" o_rpy="0 0 0" />
     </link>
-    <link name="lidar_link">
-        <visual>
-            <geometry>
-                <cylinder radius="${lidar_radius}" length="${lidar_height}" />
-            </geometry>
-            <origin xyz="0 0 ${lidar_height / 2.0}" rpy="0 0 0" />
-            <material name="green">
-                <color rgba="0 0.8 0 1" />
-            </material>
-        </visual>
-        <collision>
-            <geometry>
-                <cylinder radius="${lidar_radius}" length="${lidar_height}" />
-            </geometry>
-            <origin xyz="0 0 ${lidar_height / 2.0}" rpy="0 0 0" />
-        </collision>
-        <xacro:cylinder_inertia m="0.2" r="${lidar_radius}" l="${lidar_height}"
-                                o_xyz="0 0 ${lidar_height / 2.0}" o_rpy="0 0 0" />
-    </link>
     <joint name="base_joint" type="fixed">
         <parent link="base_footprint" />
@@ -105,8 +84,3 @@
         <origin xyz="${base_length / 3.0} 0 ${-wheel_radius / 2.0}" rpy="0 0 0" />
     </joint>
-    <joint name="base_lidar_joint" type="fixed">
-        <parent link="base_link" />
-        <child link="lidar_link" />
-        <origin xyz="0 0 ${base_height}" rpy="0 0 0" />
-    </joint>
 </robot>

File: src/sum2026_description/urdf/sum2026.urdf.xacro (robot description, xacro)
@@ -4,4 +4,5 @@
     <xacro:include filename="common_properties.xacro" />
     <xacro:include filename="mobile_base.xacro" />
+    <xacro:include filename="lidar.xacro" />
     <xacro:if value="$(arg use_sim)">
         <ros2_control name="sum2026" type="system">
@@ -24,27 +25,4 @@
             <mu2 value="0.1" />
         </gazebo>
-        <gazebo reference="lidar_link">
-            <sensor name="lidar" type="gpu_lidar">
-                <topic>scan</topic>
-                <update_rate>10</update_rate>
-                <lidar>
-                    <scan>
-                        <horizontal>
-                            <samples>360</samples>
-                            <resolution>1</resolution>
-                            <min_angle>-${pi}</min_angle>
-                            <max_angle>${pi}</max_angle>
-                        </horizontal>
-                    </scan>
-                    <range>
-                        <min>0.12</min>
-                        <max>10.0</max>
-                        <resolution>0.01</resolution>
-                    </range>
-                </lidar>
-                <always_on>true</always_on>
-                <visualize>true</visualize>
-            </sensor>
-        </gazebo>
         <gazebo>
             <plugin filename="gz_ros2_control-system" name="gz_ros2_control::GazeboSimROS2ControlPlugin">
