Commit message: feat: armじゃまだからけした

File: src/sum2026_description/urdf/common_properties.xacro (robot description, xacro)
@@ -6,10 +6,4 @@
     <material name="grey">
         <color rgba="0.5 0.5 0.5 1" />
-    </material>
-    <material name="orange">
-        <color rgba="1.0 0.5 0 1" />
-    </material>
-    <material name="yellow">
-        <color rgba="1.0 1.0 0 1" />
     </material>
     <xacro:macro name="box_inertia" params="m x y z o_xyz o_rpy">

File: src/sum2026_description/urdf/sum2026.urdf.xacro (robot description, xacro)
@@ -4,10 +4,4 @@
     <xacro:include filename="common_properties.xacro" />
     <xacro:include filename="mobile_base.xacro" />
-    <xacro:include filename="arm.xacro" />
-    <joint name="mobile_base_arm_joint" type="fixed">
-        <parent link="base_link" />
-        <child link="arm_base_link" />
-        <origin xyz="${base_length / 4.0} 0 ${base_height}" rpy="0 0 0" />
-    </joint>
     <xacro:if value="$(arg use_sim)">
         <ros2_control name="sum2026" type="system">
@@ -25,12 +19,4 @@
                 <state_interface name="velocity" />
             </joint>
-            <joint name="arm_joint1">
-                <command_interface name="position" />
-                <state_interface name="position" />
-            </joint>
-            <joint name="arm_joint2">
-                <command_interface name="position" />
-                <state_interface name="position" />
-            </joint>
         </ros2_control>
         <gazebo reference="caster_wheel_link">

Commit message: feat: lidarの色をcommon_propertiesにいれた

File: src/sum2026_description/urdf/common_properties.xacro (robot description, xacro)
@@ -6,4 +6,7 @@
     <material name="grey">
         <color rgba="0.5 0.5 0.5 1" />
+    </material>
+    <material name="green">
+        <color rgba="0 0.8 0 1" />
     </material>
     <xacro:macro name="box_inertia" params="m x y z o_xyz o_rpy">

File: src/sum2026_description/urdf/lidar.xacro (robot description, xacro)
@@ -16,7 +16,5 @@
             </geometry>
             <origin xyz="0 0 ${lidar_height / 2.0}" rpy="0 0 0" />
-            <material name="green">
-                <color rgba="0 0.8 0 1" />
-            </material>
+            <material name="green" />
         </visual>
         <collision>
